Commit message: load_gazebo_table.launch

File: birl_baxter_pnp_sim/model/tables.xacro (robot description, xacro)
@@ -2,8 +2,8 @@
 <robot name="table" xmlns:xacro="http://www.ros.org/wiki/xacro">
 <xacro:arg name="table_front" default="true"/>
-<xacro:arg name="table_right_side" default="true"/>
-<xacro:arg name="container" default="false"/>
+<!--<xacro:arg name="table_right_side" default="true"/>
+<xacro:arg name="container" default="false"/>-->
 <!-- Container -->
-<xacro:if value="$(arg container)">
+<!--<xacro:if value="$(arg container)">
 <xacro:include filename="$(find birl_baxter_description)/urdf/box/container/container.xacro">
 </xacro:include>
@@ -13,16 +13,16 @@
     <child link="container"/>
 </joint>
-</xacro:if>
+</xacro:if>   -->
 <!-- Table -->
 <xacro:if value="$(arg table_front)">
-<xacro:include filename="$(find birl_baxter_description)/urdf/table/table_front.xacro">
+<xacro:include filename="$(find birl_baxter_description)/urdf/table/table.xacro">
 </xacro:include>
 <joint name="table_fixed_1" type="fixed">
     <origin rpy="0 0 0" xyz="0.0 0.0 -0.93"/>
     <parent link="world"/>
-    <child link="table_front"/>
+    <child link="table"/>
 </joint>
 </xacro:if>
-<xacro:if value="$(arg table_right_side)">
+<!--<xacro:if value="$(arg table_right_side)">
 <xacro:include filename="$(find birl_baxter_description)/urdf/table/table_right_side.xacro">
 </xacro:include>
@@ -32,4 +32,4 @@
     <child link="table_right_side"/>
 </joint>
-</xacro:if>
+</xacro:if>-->
 </robot>
