Commit message: loading gazebo model

File: birl_baxter_pnp_sim/model/table_right_side.xacro (robot description, xacro)
@@ -1,9 +1,5 @@
 <?xml version="1.0" ?>
-<!-- =================================================================================== -->
-<!-- |    This document was autogenerated by xacro from table.xacro                    | -->
-<!-- |    EDITING THIS FILE BY HAND IS NOT RECOMMENDED                                 | -->
-<!-- =================================================================================== -->
-<robot name="table" xmlns:xacro="http://www.ros.org/wiki/xacro">
-  <link name="table">
+<robot name="table_right_side" xmlns:xacro="http://www.ros.org/wiki/xacro">
+  <link name="table_right_side">
     <visual>
       <origin rpy="0 0 0" xyz="0.6 0 0"/>
@@ -24,10 +20,5 @@
     </inertial>
   </link>
-  <!-- <joint name="table_fixed" type="fixed">
-    <origin rpy="0 0 0" xyz="0.0 0.0 -0.93"/>
-    <parent link="base"/>
-    <child link="table"/>
-  </joint>-->
-  <gazebo reference="table">
+  <gazebo reference="table_right_side">
     <self_collide>1</self_collide>
     <mu1>1000000</mu1>
