Commit message: last saving

File: birl_baxter_pnp_sim/model/gazebo_env_setup.xacro (robot description, xacro)
@@ -4,4 +4,5 @@
   <xacro:arg name="table_right_side" default="true"/>
   <xacro:arg name="container" default="true"/>
+  <xacro:arg name="picking_box" default="false"/>
    <link name="world">
 </link>
@@ -11,5 +12,5 @@
     </xacro:include>
     <joint name="table_fixed_1" type="fixed">
-      <origin rpy="0 0 0" xyz="0.0 0.0 -0.93"/>
+      <origin rpy="0 0 0" xyz="0.6 0.0 0.0"/>
       <parent link="world"/>
       <child link="table_front"/>
@@ -21,5 +22,5 @@
     </xacro:include>
     <joint name="table_fixed_2" type="fixed">
-      <origin rpy="0 0 -1.57" xyz="0.0 -0.2 -0.93"/>
+      <origin rpy="0 0 -1.57" xyz="0.4 -0.85 0.0"/>
       <parent link="world"/>
       <child link="table_right_side"/>
@@ -31,8 +32,18 @@
     </xacro:include>
     <joint name="container_fixed" type="fixed">
-      <origin rpy="0 0 0" xyz="-0.1 -0.95 -0.13"/>
+      <origin rpy="0 0 -1.57" xyz="0.1 -0.70 0.81"/>
       <parent link="world"/>
       <child link="container"/>
     </joint>
   </xacro:if>
+      <!-- picking_box-->
+  <xacro:if value="$(arg picking_box)">
+    <xacro:include filename="$(find birl_baxter_pnp_sim)/model/picking_box.xacro">
+    </xacro:include>
+    <joint name="picking_box_fixed" type="fixed">
+      <origin rpy="0 0 0" xyz="-0.07 -0.9 0.8"/>
+      <parent link="world"/>
+      <child link="picking_box"/>
+    </joint>
+  </xacro:if>
 </robot>

File: birl_baxter_pnp_sim/model/picking_box.xacro (robot description, xacro)
@@ -1,9 +1,9 @@
 <?xml version="1.0" ?>
-<robot name="table_front" xmlns:xacro="http://www.ros.org/wiki/xacro">
-  <link name="table_front">
+<robot name="picking_box" xmlns:xacro="http://www.ros.org/wiki/xacro">
+  <link name="picking_box">
     <visual>
       <origin rpy="0 0 0" xyz="0 0 0"/>
       <geometry>
-        <mesh filename="package://birl_baxter_description/meshes/table/table.dae"/>
+        <mesh filename="package://birl_baxter_description/urdf/box/picking_box/picking_box.STL"/>
       </geometry>
     </visual>
@@ -11,14 +11,14 @@
       <origin rpy="0 0 0" xyz="0 0 0"/>
       <geometry>
-        <mesh filename="package://birl_baxter_description/meshes/table/table.stl"/>
+        <mesh filename="package://birl_baxter_description/urdf/box/picking_box/picking_box.STL"/>
       </geometry>
     </collision>
     <inertial>
       <origin rpy="0 0 0" xyz="0 0 0"/>
-      <mass value="60.86397744"/>
-      <inertia ixx="5.0635929" ixy="0.00103417" ixz="0.80199628" iyy="6.08689388" iyz="0.00105311" izz="4.96191932"/>
+      <mass value="0.05"/>
+      <inertia ixx="0.001" ixy="0.00103417" ixz="0.80199628" iyy="6.08689388" iyz="0.00105311" izz="4.96191932"/>
     </inertial>
   </link>
-  <gazebo reference="table_front">
+  <gazebo reference="picking_box">
     <self_collide>1</self_collide>
     <mu1>1000000</mu1>

File: birl_baxter_pnp_sim/model/table_right_side.xacro (robot description, xacro)
@@ -3,5 +3,5 @@
   <link name="table_right_side">
     <visual>
-      <origin rpy="0 0 0" xyz="0.6 0 0"/>
+      <origin rpy="0 0 0" xyz="0.0 -0.2 0"/>
       <geometry>
         <mesh filename="package://birl_baxter_description/meshes/table/table.dae"/>
@@ -9,5 +9,5 @@
     </visual>
     <collision>
-      <origin rpy="0 0 0" xyz="0.6 0 0"/>
+      <origin rpy="0 0 0" xyz="0.0 -0.2 0"/>
       <geometry>
         <mesh filename="package://birl_baxter_description/meshes/table/table.stl"/>
@@ -15,5 +15,5 @@
     </collision>
     <inertial>
-      <origin rpy="0 0 0" xyz="0.6 0 0"/>
+      <origin rpy="0 0 0" xyz="0.0 -0.2 0"/>
       <mass value="60.86397744"/>
       <inertia ixx="5.0635929" ixy="0.00103417" ixz="0.80199628" iyy="6.08689388" iyz="0.00105311" izz="4.96191932"/>
