Commit message: save

File: birl_baxter_pnp_sim/model/container.xacro (robot description, xacro)
@@ -5,5 +5,5 @@
       <origin rpy="0 0 0" xyz="0 0 0"/>
       <geometry>
-        <mesh filename="package://birl_baxter_description/meshes/container/container.STL"/>
+        <mesh filename="package://birl_baxter_description/meshes/container/container.stl"/>
       </geometry>
     </visual>
@@ -11,5 +11,5 @@
       <origin rpy="0 0 0" xyz="0 0 0"/>
       <geometry>
-        <mesh filename="package://birl_baxter_description/meshes/container/container.STL"/>
+        <mesh filename="package://birl_baxter_description/meshes/container/container.stl"/>
       </geometry>
     </collision>
